Commit message: Updated meshes, added yaml support for controller

File: bin/optitrack/resources/model/HRP4c.urdf (robot description, URDF)
Before this commit: robot HRP4C, 37 links, 36 joints
Links:
- link LL_KOSY_L1: mass 2.7752200000 -> 1
- link LL_KOSY_L23: mass 2.2450500000 -> 1
- link LL_KOSY_L4: mass 2.6274500000 -> 1; geometry visual mesh filename=../../../model/HRP4c/graphics/L_HIP_P_rev2.obj
- link LL_KOSY_L56: mass 5.7035400000 -> 1; geometry visual mesh filename=../../../model/HRP4c/graphics/L_KNEE_P_rev2.obj
- link LL_ankle: mass 0.3906700000 -> 1
- link LL_foot: mass 1.4241951000 -> 1
- link RL_KOSY_L23: mass 2.2450500000 -> 1
- link RL_KOSY_L4: mass 2.6274500000 -> 1; geometry visual mesh filename=../../../model/HRP4c/graphics/R_HIP_P_rev2.obj
- link RL_KOSY_L56: mass 5.7035400000 -> 1; geometry visual mesh filename=../../../model/HRP4c/graphics/R_KNEE_P_rev2.obj
- link RL_ankle: mass 0.3906700000 -> 1
- link RL_foot: mass 1.4241951000 -> 1; geometry visual mesh filename=../../../model/HRP4c/graphics/R_ANKLE_R_rev2.obj
- link hip_base: mass 5.6174600000 -> 1
- link la_end_effector: mass 0.1 -> 1
- link la_link1: mass 2.2396100000 -> 1
- link la_link3: mass 2.3629100000 -> 1; geometry visual mesh filename=../../../model/HRP4c/graphics/L_SHOULDER_Y_rev2.obj
- link la_link4: mass 0.7187000000 -> 1; geometry visual mesh filename=../../../model/HRP4c/graphics/L_ELBOW_P_rev2.obj
- link la_link5: mass 2.2786200000 -> 1
- link la_link6: mass 0.2863747200 -> 1
- link neck_link1: mass 0.3364400000 -> 1
- link neck_link2: mass 2.4522900000 -> 1; geometry visual mesh filename=../../../model/HRP4c/graphics/Helmet_roboCop_rev2.obj; visual mesh filename=../../../model/HRP4c/graphics/NECK_P.obj
- link ra_end_effector: mass 0.1 -> 1; geometry visual mesh filename=../../../model/HRP4c/graphics/R_WRIST_R_rev2.obj
- link ra_link1: mass 2.2396100000 -> 1
- link ra_link2: mass 1.0993800000 -> 1
- link ra_link3: mass 2.3629100000 -> 1; geometry visual mesh filename=../../../model/HRP4c/graphics/R_SHOULDER_Y_rev2.obj
- link ra_link4: mass 0.7187000000 -> 1; geometry visual mesh filename=../../../model/HRP4c/graphics/R_ELBOW_P_rev2.obj
- link ra_link5: mass 2.2786200000 -> 1; geometry visual mesh filename=../../../model/HRP4c/graphics/R_WRIST_Y_rev2.obj
- link ra_link6: mass 0.2863747200 -> 1
- link trunk: mass 18.9794300000 -> 1
- link trunk_rz: mass 18.9794300000 -> 1; geometry visual mesh filename=../../../model/HRP4c/graphics/CHEST_Y2_rev2.obj
Joints:
- joint floating_base_r1: limit lower=-5.00 upper=5.00 effort=4000 velocity=1000 -> lower=-1000.00 upper=1000.00 effort=4000 velocity=1000
- joint floating_base_r2: limit lower=-5.00 upper=5.00 effort=4000 velocity=1000 -> lower=-1000.00 upper=1000.00 effort=4000 velocity=1000
- joint floating_base_r3: limit lower=-5.00 upper=5.00 effort=4000 velocity=1000 -> lower=-1000.00 upper=1000.00 effort=4000 velocity=1000
- joint j1: limit lower=-3.1415 upper=3.1415 effort=176 velocity=1.9199 -> lower=-0.3 upper=0.3 effort=176 velocity=1.9199
- joint j11: limit lower=-3.1415 upper=3.1415 effort=50 velocity=2.0944 -> lower=-1 upper=1 effort=50 velocity=2.0944
- joint j12: limit lower=-3.1415 upper=3.1415 effort=165 velocity=3.0718 -> lower=-0.8 upper=0.8 effort=165 velocity=3.0718
- joint j13: limit lower=-3.1415 upper=3.1415 effort=100 velocity=2.7402 -> lower=-0.1 upper=0.1 effort=100 velocity=2.7402
- joint j14: limit lower=-3.1415 upper=3.1415 effort=100 velocity=2.7402 -> lower=-0.8 upper=0.8 effort=100 velocity=2.7402
- joint j15: limit lower=-3.1415 upper=3.1415 effort=100 velocity=2.7402 -> lower=-3.1415 upper=0.4 effort=100 velocity=2.7402
- joint j16: limit lower=-3.1415 upper=-0.2 effort=100 velocity=2.7402 -> lower=-2.8 upper=-0.1 effort=100 velocity=2.7402
- joint j17: limit lower=-3.1415 upper=3.1415 effort=40 velocity=2.0944 -> lower=-1 upper=1 effort=40 velocity=2.0944
- joint j18: limit lower=-3.1415 upper=-0.05 effort=40 velocity=2.0944 -> lower=-3.1415 upper=-0.1 effort=40 velocity=2.0944
- joint j19: limit lower=-3.1415 upper=3.1415 effort=40 velocity=2.0944 -> lower=-1.0 upper=1.0 effort=40 velocity=2.0944
- joint j2: limit lower=-3.1415 upper=3.1415 effort=100 velocity=2.7402 -> lower=-1.5717 upper=1.5717 effort=100 velocity=2.7402
- joint j20: limit lower=-3.1415 upper=3.1415 effort=35 velocity=2.0944 -> lower=-0.3 upper=1.4 effort=35 velocity=2.0944
- joint j22: limit lower=0.2 upper=3.1415 effort=100 velocity=2.7402 -> lower=0.1 upper=2.8 effort=100 velocity=2.7402
- joint j23: limit lower=-3.1415 upper=3.1415 effort=40 velocity=2.0944 -> lower=-1 upper=1 effort=40 velocity=2.0944
- joint j24: limit lower=-3.1415 upper=-0.05 effort=40 velocity=2.0944 -> lower=-3.1415 upper=-0.1 effort=40 velocity=2.0944
- joint j25: limit lower=-3.1415 upper=3.1415 effort=40 velocity=2.0944 -> lower=-1.0 upper=1.0 effort=40 velocity=2.0944
- joint j26: limit lower=-3.1415 upper=3.1415 effort=40 velocity=2.0944 -> lower=-0.3 upper=1.4 effort=40 velocity=2.0944
- joint j27: limit lower=-3.1415 upper=3.1415 effort=8.4 velocity=4.7124 -> lower=-0.8 upper=0.8 effort=8.4 velocity=4.7124
- joint j28: limit lower=-3.1415 upper=3.1415 effort=8.4 velocity=4.7124 -> lower=-1 upper=0.2 effort=8.4 velocity=4.7124
- joint j4: limit lower=0.5 upper=3.1415 effort=165 velocity=3.0718 -> lower=0.1 upper=3.1415 effort=165 velocity=3.0718
- joint j5: limit lower=-3.1415 upper=3.1415 effort=50 velocity=2.0944 -> lower=-1 upper=1 effort=50 velocity=2.0944
- joint j6: limit lower=-3.1415 upper=3.1415 effort=165 velocity=3.0718 -> lower=-0.8 upper=0.8 effort=165 velocity=3.0718
- joint j7: limit lower=-3.1415 upper=3.1415 effort=176 velocity=1.9199 -> lower=-0.3 upper=0.3 effort=176 velocity=1.9199
- joint j8: limit lower=-3.1415 upper=3.1415 effort=100 velocity=2.7402 -> lower=-1.5717 upper=1.5717 effort=100 velocity=2.7402
- joint j_lhand_revolute: limit lower=-3.1415 upper=3.1415 effort=35 velocity=2.0944 -> lower=-0.9 upper=0.3 effort=35 velocity=2.0944
- joint j_rhand_revolute: limit lower=-3.1415 upper=3.1415 effort=35 velocity=2.0944 -> lower=-0.9 upper=0.3 effort=35 velocity=2.0944
