Commit message: Minor updates

File: optitrack/model/HRP4c.urdf (robot description, URDF)
Before this commit: robot HRP4C, 37 links, 36 joints
Joints:
- joint floating_base_p1: limit lower=-5.00 upper=5.00 effort=4000 velocity=1000 -> lower=-100.00 upper=100.00 effort=4000 velocity=1000
- joint floating_base_p2: limit lower=-5.00 upper=5.00 effort=4000 velocity=1000 -> lower=-100.00 upper=100.00 effort=4000 velocity=1000
- joint floating_base_p3: limit lower=-5.00 upper=5.00 effort=4000 velocity=1000 -> lower=-100.00 upper=100.00 effort=4000 velocity=1000
- joint floating_base_r1: limit lower=-1000.00 upper=1000.00 effort=4000 velocity=1000 -> lower=-1000000.00 upper=1000000.00 effort=4000 velocity=1000
- joint floating_base_r2: limit lower=-1000.00 upper=1000.00 effort=4000 velocity=1000 -> lower=-1000000.00 upper=1000000.00 effort=4000 velocity=1000
- joint floating_base_r3: limit lower=-1000.00 upper=1000.00 effort=4000 velocity=1000 -> lower=-1000000.00 upper=1000000.00 effort=4000 velocity=1000

Commit message: Post October 6 test

File: optitrack/model/HRP4c.urdf (robot description, URDF)
Before this commit: robot HRP4c, 37 links, 36 joints
Joints:
- joint j1: limit lower=-0.3 upper=0.3 effort=176 velocity=1.9199 -> lower=-0.8 upper=0.8 effort=176 velocity=1.9199
- joint j10: limit lower=0.5 upper=3.1415 effort=165 velocity=3.0718 -> lower=0.1 upper=2.5 effort=165 velocity=3.0718
- joint j11: limit lower=-1 upper=1 effort=50 velocity=2.0944 -> lower=-0.5 upper=0.5 effort=50 velocity=2.0944
- joint j12: limit lower=-0.8 upper=0.8 effort=165 velocity=3.0718 -> lower=-0.6 upper=0.6 effort=165 velocity=3.0718
- joint j13: limit lower=-0.1 upper=0.1 effort=100 velocity=2.7402 -> lower=-0.5 upper=1.5717 effort=100 velocity=2.7402
- joint j15: limit lower=-3.1415 upper=0.4 effort=100 velocity=2.7402 -> lower=-3.1415 upper=0.6 effort=100 velocity=2.7402
- joint j16: limit lower=-2.8 upper=-0.1 effort=100 velocity=2.7402 -> lower=-3.1415 upper=0.8 effort=100 velocity=2.7402
- joint j17: limit lower=-1 upper=1 effort=40 velocity=2.0944 -> lower=-0.5 upper=0.5 effort=40 velocity=2.0944
- joint j19: limit lower=-1.0 upper=1.0 effort=40 velocity=2.0944 -> lower=-0.5 upper=0.5 effort=40 velocity=2.0944
- joint j21: limit lower=-3.1415 upper=3.1415 effort=100 velocity=2.7402 -> lower=-3.1415 upper=0.6 effort=100 velocity=2.7402
- joint j22: limit lower=0.1 upper=2.8 effort=100 velocity=2.7402 -> lower=-0.8 upper=3.1415 effort=100 velocity=2.7402
- joint j23: limit lower=-1 upper=1 effort=40 velocity=2.0944 -> lower=-0.5 upper=0.5 effort=40 velocity=2.0944
- joint j25: limit lower=-1.0 upper=1.0 effort=40 velocity=2.0944 -> lower=-0.5 upper=0.5 effort=40 velocity=2.0944
- joint j3: limit lower=-3.1415 upper=3.1415 effort=100 velocity=2.7402 -> lower=-1.5717 upper=1.5717 effort=100 velocity=2.7402
- joint j4: limit lower=0.1 upper=3.1415 effort=165 velocity=3.0718 -> lower=0.1 upper=2.5 effort=165 velocity=3.0718
- joint j5: limit lower=-1 upper=1 effort=50 velocity=2.0944 -> lower=-0.5 upper=0.5 effort=50 velocity=2.0944
- joint j6: limit lower=-0.8 upper=0.8 effort=165 velocity=3.0718 -> lower=-0.6 upper=0.6 effort=165 velocity=3.0718
- joint j7: limit lower=-0.3 upper=0.3 effort=176 velocity=1.9199 -> lower=-0.8 upper=0.8 effort=176 velocity=1.9199
- joint j9: limit lower=-3.1415 upper=3.1415 effort=100 velocity=2.7402 -> lower=-1.5717 upper=1.5717 effort=100 velocity=2.7402

Commit message: Tuned setup; investigate joint limits

File: optitrack/model/HRP4c.urdf (robot description, URDF)
Before this commit: robot HRP4c, 37 links, 36 joints
Links:
- link la_end_effector: geometry visual mesh filename=../../../model/HRP4c/graphics/L_WRIST_R.obj; visual sphere radius=0.05
- link ra_end_effector: geometry visual mesh filename=../../../model/HRP4c/graphics/R_WRIST_R_rev2.obj; visual sphere radius=0.05
Joints:
- joint j18: limit lower=-3.1415 upper=-0.1 effort=40 velocity=2.0944 -> lower=-3.1415 upper=-0.5 effort=40 velocity=2.0944
- joint j24: limit lower=-3.1415 upper=-0.1 effort=40 velocity=2.0944 -> lower=-3.1415 upper=-0.5 effort=40 velocity=2.0944

Commit message: Post session, untested change removing elbow tracking and sent to posture task; need to confirm

File: optitrack/model/HRP4c.urdf (robot description, URDF)
Before this commit: robot HRP4c, 37 links, 36 joints
Links:
- link la_end_effector: geometry visual mesh filename=../../../model/HRP4c/graphics/L_WRIST_R.obj
- link ra_end_effector: geometry visual mesh filename=../../../model/HRP4c/graphics/R_WRIST_R_rev2.obj

Commit message: Tuned controller with combined pos/ori and proper reduced-rank orientation setup; need to test with operator

File: optitrack/model/HRP4c.urdf (robot description, URDF)
Before this commit: robot HRP4c, 37 links, 36 joints
Links:
- added link LL_ankle_2, mass 1.0
- added link RL_ankle_2, mass 1.0
- link RL_KOSY_L1: mass 2.7752200000 -> 1
- link trunk_rz: mass 1 -> 100
Joints:
- added joint j_11.5: type revolute, parent LL_ankle, child LL_ankle_2, origin xyz=0.0 0.0 0.0 rpy=0.0 0.0 0.0, axis 0.0 0.0 1.0, limit lower=-0.5 upper=0.5 effort=50.0 velocity=50.0
- added joint j_5.5: type revolute, parent RL_ankle, child RL_ankle_2, origin xyz=0.0 0.0 0.0 rpy=0.0 0.0 0.0, axis 0.0 0.0 1.0, limit lower=-0.5 upper=0.5 effort=50.0 velocity=50.0
- joint j12: parent LL_ankle -> LL_ankle_2
- joint j25: origin xyz=0.0000 0.035  -0.21 rpy=0.177 0 0 -> xyz=0.0000 0.035 -0.21 rpy=0.177 0 0
- joint j6: parent RL_ankle -> RL_ankle_2
- joint j_lhand_revolute: axis 1 0 0 -> 0 0 1
- joint j_rhand_revolute: axis 1 0 0 -> 0 0 1

Commit message: October 15 fine tuned; need to test offline data and robustness

File: optitrack/model/HRP4c.urdf (robot description, URDF)
Before this commit: robot HRP4c, 39 links, 38 joints
Links:
- link LL_KOSY_L56: geometry visual mesh filename=../../../model/HRP4c/graphics/L_KNEE_P_rev2.obj; visual sphere radius=0.05

Commit message: Added collision meshes; might need to tune hands

File: optitrack/model/HRP4c.urdf (robot description, URDF)
Before this commit: robot HRP4c, 39 links, 38 joints
Links:
- link LL_KOSY_L4: geometry collision cylinder length=0.25 radius=0.05; visual mesh filename=../../../model/HRP4c/graphics/L_HIP_P_rev2.obj
- link LL_KOSY_L56: geometry collision cylinder length=0.2 radius=0.05; visual mesh filename=../../../model/HRP4c/graphics/L_KNEE_P_rev2.obj
- link LL_foot: geometry collision sphere radius=0.03; visual mesh filename=../../../model/HRP4c/graphics/L_ANKLE_R.obj
- link RL_KOSY_L4: geometry collision cylinder length=0.25 radius=0.05; visual mesh filename=../../../model/HRP4c/graphics/R_HIP_P_rev2.obj
- link RL_KOSY_L56: geometry collision cylinder length=0.2 radius=0.05; visual mesh filename=../../../model/HRP4c/graphics/R_KNEE_P_rev2.obj
- link RL_foot: geometry collision sphere radius=0.03; visual mesh filename=../../../model/HRP4c/graphics/R_ANKLE_R_rev2.obj
- link la_end_effector: geometry collision sphere radius=0.05; visual mesh filename=../../../model/HRP4c/graphics/L_WRIST_R.obj
- link la_link3: geometry collision cylinder length=0.15 radius=0.04; visual mesh filename=../../../model/HRP4c/graphics/L_SHOULDER_Y_rev2.obj
- link la_link5: geometry collision cylinder length=0.13 radius=0.04; visual mesh filename=../../../model/HRP4c/graphics/L_WRIST_Y.obj
- link neck_link2: geometry collision sphere radius=0.12; visual mesh filename=../../../model/HRP4c/graphics/Helmet_roboCop_rev2.obj
- link ra_end_effector: geometry collision sphere radius=0.05; visual mesh filename=../../../model/HRP4c/graphics/R_WRIST_R_rev2.obj
- link ra_link3: geometry collision cylinder length=0.15 radius=0.04; visual mesh filename=../../../model/HRP4c/graphics/R_SHOULDER_Y_rev2.obj
- link ra_link5: geometry collision cylinder length=0.13 radius=0.04; visual mesh filename=../../../model/HRP4c/graphics/R_WRIST_Y_rev2.obj
- link trunk_rz: geometry collision cylinder length=0.45 radius=0.13; visual mesh filename=../../../model/HRP4c/graphics/CHEST_Y2_rev2.obj

File: optitrack/model/HRP4c_green.urdf (robot description, URDF)
Before this commit: robot HRP4c, 39 links, 38 joints
Links:
- link LL_KOSY_L4: geometry collision cylinder length=0.25 radius=0.05; visual mesh filename=../../../model/HRP4c/graphics/L_HIP_P_rev2.obj
- link LL_KOSY_L56: geometry collision cylinder length=0.2 radius=0.05; visual mesh filename=../../../model/HRP4c/graphics/L_KNEE_P_rev2.obj
- link LL_foot: geometry collision sphere radius=0.03; visual mesh filename=../../../model/HRP4c/graphics/L_ANKLE_R.obj
- link RL_KOSY_L4: geometry collision cylinder length=0.25 radius=0.05; visual mesh filename=../../../model/HRP4c/graphics/R_HIP_P_rev2.obj
- link RL_KOSY_L56: geometry collision cylinder length=0.2 radius=0.05; visual mesh filename=../../../model/HRP4c/graphics/R_KNEE_P_rev2.obj
- link RL_foot: geometry collision sphere radius=0.03; visual mesh filename=../../../model/HRP4c/graphics/R_ANKLE_R_rev2.obj
- link la_end_effector: geometry collision sphere radius=0.05; visual mesh filename=../../../model/HRP4c/graphics/L_WRIST_R.obj
- link la_link3: geometry collision cylinder length=0.15 radius=0.04; visual mesh filename=../../../model/HRP4c/graphics/L_SHOULDER_Y_rev2.obj
- link la_link5: geometry collision cylinder length=0.13 radius=0.04; visual mesh filename=../../../model/HRP4c/graphics/L_WRIST_Y.obj
- link neck_link2: geometry collision sphere radius=0.12; visual mesh filename=../../../model/HRP4c/graphics/Helmet_roboCop_rev2_green.obj
- link ra_end_effector: geometry collision sphere radius=0.05; visual mesh filename=../../../model/HRP4c/graphics/R_WRIST_R_rev2.obj
- link ra_link3: geometry collision cylinder length=0.15 radius=0.04; visual mesh filename=../../../model/HRP4c/graphics/R_SHOULDER_Y_rev2.obj
- link ra_link5: geometry collision cylinder length=0.13 radius=0.04; visual mesh filename=../../../model/HRP4c/graphics/R_WRIST_Y_rev2.obj
- link trunk_rz: geometry collision cylinder length=0.45 radius=0.13; visual mesh filename=../../../model/HRP4c/graphics/CHEST_Y2_rev2.obj

File: optitrack/model/HRP4c_purple.urdf (robot description, URDF)
Before this commit: robot HRP4c, 39 links, 38 joints
Links:
- link LL_KOSY_L4: geometry collision cylinder length=0.25 radius=0.05; visual mesh filename=../../../model/HRP4c/graphics/L_HIP_P_rev2.obj
- link LL_KOSY_L56: geometry collision cylinder length=0.2 radius=0.05; visual mesh filename=../../../model/HRP4c/graphics/L_KNEE_P_rev2.obj
- link LL_foot: geometry collision sphere radius=0.03; visual mesh filename=../../../model/HRP4c/graphics/L_ANKLE_R.obj
- link RL_KOSY_L4: geometry collision cylinder length=0.25 radius=0.05; visual mesh filename=../../../model/HRP4c/graphics/R_HIP_P_rev2.obj
- link RL_KOSY_L56: geometry collision cylinder length=0.2 radius=0.05; visual mesh filename=../../../model/HRP4c/graphics/R_KNEE_P_rev2.obj
- link RL_foot: geometry collision sphere radius=0.03; visual mesh filename=../../../model/HRP4c/graphics/R_ANKLE_R_rev2.obj
- link la_end_effector: geometry collision sphere radius=0.05; visual mesh filename=../../../model/HRP4c/graphics/L_WRIST_R.obj
- link la_link3: geometry collision cylinder length=0.15 radius=0.04; visual mesh filename=../../../model/HRP4c/graphics/L_SHOULDER_Y_rev2.obj
- link la_link5: geometry collision cylinder length=0.13 radius=0.04; visual mesh filename=../../../model/HRP4c/graphics/L_WRIST_Y.obj
- link neck_link2: geometry collision sphere radius=0.12; visual mesh filename=../../../model/HRP4c/graphics/Helmet_roboCop_rev2_purple.obj
- link ra_end_effector: geometry collision sphere radius=0.05; visual mesh filename=../../../model/HRP4c/graphics/R_WRIST_R_rev2.obj
- link ra_link3: geometry collision cylinder length=0.15 radius=0.04; visual mesh filename=../../../model/HRP4c/graphics/R_SHOULDER_Y_rev2.obj
- link ra_link5: geometry collision cylinder length=0.13 radius=0.04; visual mesh filename=../../../model/HRP4c/graphics/R_WRIST_Y_rev2.obj
- link trunk_rz: geometry collision cylinder length=0.45 radius=0.13; visual mesh filename=../../../model/HRP4c/graphics/CHEST_Y2_rev2.obj
