Commit message: Tuned after Oct 11; need to change upper leg socket to spherical

File: optitrack/model/HRP4c_green.urdf (robot description, URDF)
Before this commit: robot HRP4c, 37 links, 36 joints
Links:
- link neck_link2: geometry visual mesh filename=../../../model/HRP4c/graphics/Helmet_roboCop_rev2_green.obj; visual mesh filename=../../../model/HRP4c/graphics/NECK_P.obj

File: optitrack/model/HRP4c_purple.urdf (robot description, URDF)
Before this commit: robot HRP4c, 37 links, 36 joints
Links:
- link neck_link2: geometry visual mesh filename=../../../model/HRP4c/graphics/Helmet_roboCop_rev2_purple.obj; visual mesh filename=../../../model/HRP4c/graphics/NECK_P.obj

Commit message: Revised 2 dancer simulation and type 1 singularity enabling

File: optitrack/model/HRP4c_green.urdf (robot description, URDF)
Before this commit: robot HRP4c, 37 links, 36 joints
Links:
- added link LL_ankle_2, mass 1.0
- added link RL_ankle_2, mass 1.0
- link LL_KOSY_L56: geometry visual mesh filename=../../../model/HRP4c/graphics/L_KNEE_P_rev2.obj; visual sphere radius=0.05
- link RL_KOSY_L1: mass 2.7752200000 -> 1
- link trunk_rz: mass 1 -> 100
Joints:
- added joint j_11.5: type revolute, parent LL_ankle, child LL_ankle_2, origin xyz=0.0 0.0 0.0 rpy=0.0 0.0 0.0, axis 0.0 0.0 1.0, limit lower=-0.5 upper=0.5 effort=50.0 velocity=50.0
- added joint j_5.5: type revolute, parent RL_ankle, child RL_ankle_2, origin xyz=0.0 0.0 0.0 rpy=0.0 0.0 0.0, axis 0.0 0.0 1.0, limit lower=-0.5 upper=0.5 effort=50.0 velocity=50.0
- joint j12: parent LL_ankle -> LL_ankle_2
- joint j25: origin xyz=0.0000 0.035  -0.21 rpy=0.177 0 0 -> xyz=0.0000 0.035 -0.21 rpy=0.177 0 0
- joint j6: parent RL_ankle -> RL_ankle_2
- joint j_lhand_revolute: axis 1 0 0 -> 0 0 1
- joint j_rhand_revolute: axis 1 0 0 -> 0 0 1

File: optitrack/model/HRP4c_purple.urdf (robot description, URDF)
Before this commit: robot HRP4c, 37 links, 36 joints
Links:
- added link LL_ankle_2, mass 1.0
- added link RL_ankle_2, mass 1.0
- link LL_KOSY_L56: geometry visual mesh filename=../../../model/HRP4c/graphics/L_KNEE_P_rev2.obj; visual sphere radius=0.05
- link RL_KOSY_L1: mass 2.7752200000 -> 1
- link trunk_rz: mass 1 -> 100
Joints:
- added joint j_11.5: type revolute, parent LL_ankle, child LL_ankle_2, origin xyz=0.0 0.0 0.0 rpy=0.0 0.0 0.0, axis 0.0 0.0 1.0, limit lower=-0.5 upper=0.5 effort=50.0 velocity=50.0
- added joint j_5.5: type revolute, parent RL_ankle, child RL_ankle_2, origin xyz=0.0 0.0 0.0 rpy=0.0 0.0 0.0, axis 0.0 0.0 1.0, limit lower=-0.5 upper=0.5 effort=50.0 velocity=50.0
- joint j12: parent LL_ankle -> LL_ankle_2
- joint j25: origin xyz=0.0000 0.035  -0.21 rpy=0.177 0 0 -> xyz=0.0000 0.035 -0.21 rpy=0.177 0 0
- joint j6: parent RL_ankle -> RL_ankle_2
- joint j_lhand_revolute: axis 1 0 0 -> 0 0 1
- joint j_rhand_revolute: axis 1 0 0 -> 0 0 1

Commit message: Added lpf, damping, tuned nullspace

File: optitrack/model/HRP4c_green.urdf (robot description, URDF)
Before this commit: robot HRP4c, 39 links, 38 joints
Links:
- link neck_link2: geometry collision sphere radius=0.12; visual mesh filename=../../../model/HRP4c/graphics/Helmet_roboCop_rev2.obj

File: optitrack/model/HRP4c_purple.urdf (robot description, URDF)
Before this commit: robot HRP4c, 39 links, 38 joints
Links:
- link neck_link2: geometry collision sphere radius=0.12; visual mesh filename=../../../model/HRP4c/graphics/Helmet_roboCop_rev2.obj

Commit message: pre-alumni setup

File: optitrack/model/HRP4c_green.urdf (robot description, URDF)
Before this commit: robot HRP4c, 39 links, 38 joints
Links:
- link LL_KOSY_L1: mass 1 -> 2.7752200000
- link LL_KOSY_L23: mass 1 -> 2.2450500000
- link LL_KOSY_L4: mass 1 -> 2.6274500000
- link LL_KOSY_L56: mass 1 -> 5.7035400000
- link LL_ankle: mass 1 -> 0.3906700000
- link LL_foot: mass 1 -> 1.4241951000
- link RL_KOSY_L1: mass 1 -> 2.7752200000
- link RL_KOSY_L23: mass 1 -> 2.2450500000
- link RL_KOSY_L4: mass 1 -> 2.6274500000
- link RL_KOSY_L56: mass 1 -> 5.7035400000
- link RL_foot: mass 1 -> 1.4241951000
- link hip_base: mass 1 -> 5.6174600000
- link la_link1: mass 1 -> 2.2396100000
- link la_link3: mass 1 -> 2.3629100000
- link la_link4: mass 1 -> 0.7187000000
- link la_link5: mass 1 -> 2.2786200000
- link la_link6: mass 1 -> 0.2863747200
- link ra_link1: mass 1 -> 2.2396100000
- link ra_link2: mass 1 -> 1.0993800000
- link ra_link3: mass 1 -> 2.3629100000
- link ra_link4: mass 1 -> 0.7187000000
- link ra_link5: mass 1 -> 2.2786200000
- link trunk: mass 1 -> 18.9794300000
- link trunk_rz: mass 100 -> 18.9794300000

File: optitrack/model/human.urdf (robot description, URDF)
Before this commit: robot HRP4c, 39 links, 38 joints
Links:
- link LL_KOSY_L1: mass 2.7752200000 -> 2
- link LL_KOSY_L23: mass 2.2450500000 -> 2
- link LL_KOSY_L4: mass 2.6274500000 -> 2; geometry collision cylinder length=0.25 radius=0.05; visual mesh filename=../../../model/HRP4c/graphics/L_HIP_P_rev2.obj
- link LL_KOSY_L56: mass 5.7035400000 -> 1; geometry collision cylinder length=0.2 radius=0.05; visual mesh filename=../../../model/HRP4c/graphics/L_KNEE_P_rev2.obj
- link LL_ankle: mass 0.3906700000 -> 1
- link LL_foot: mass 1.4241951000 -> 1; geometry collision sphere radius=0.03; visual mesh filename=../../../model/HRP4c/graphics/L_ANKLE_R.obj
- link RL_KOSY_L1: mass 2.7752200000 -> 2
- link RL_KOSY_L23: mass 2.2450500000 -> 2
- link RL_KOSY_L4: mass 2.6274500000 -> 2; geometry collision cylinder length=0.25 radius=0.05; visual mesh filename=../../../model/HRP4c/graphics/R_HIP_P_rev2.obj
- link RL_KOSY_L56: mass 5.7035400000 -> 1; geometry collision cylinder length=0.2 radius=0.05; visual mesh filename=../../../model/HRP4c/graphics/R_KNEE_P_rev2.obj
- link RL_ankle: mass 1 -> 0.5
- link RL_ankle_2: mass 1.0 -> 0.1
- link RL_foot: mass 1.4241951000 -> 1; geometry collision sphere radius=0.03; visual mesh filename=../../../model/HRP4c/graphics/R_ANKLE_R_rev2.obj
- link hip_base: mass 5.6174600000 -> 15
- link la_end_effector: geometry collision sphere radius=0.05; visual mesh filename=../../../model/HRP4c/graphics/L_WRIST_R.obj
- link la_link1: mass 2.2396100000 -> 1
- link la_link3: mass 2.3629100000 -> 1; geometry collision cylinder length=0.15 radius=0.04; visual mesh filename=../../../model/HRP4c/graphics/L_SHOULDER_Y_rev2.obj
- link la_link5: mass 2.2786200000 -> 1; geometry collision cylinder length=0.13 radius=0.04; visual mesh filename=../../../model/HRP4c/graphics/L_WRIST_Y.obj
- link neck_link1: mass 1 -> 2
- link neck_link2: mass 1 -> 2; geometry collision sphere radius=0.12; visual mesh filename=../../../model/HRP4c/graphics/Helmet_roboCop_rev2.obj
- link ra_end_effector: geometry collision sphere radius=0.05; visual mesh filename=../../../model/HRP4c/graphics/R_WRIST_R_rev2.obj
- link ra_link1: mass 2.2396100000 -> 1
- link ra_link3: mass 2.3629100000 -> 1; geometry collision cylinder length=0.15 radius=0.04; visual mesh filename=../../../model/HRP4c/graphics/R_SHOULDER_Y_rev2.obj
- link ra_link5: mass 2.2786200000 -> 1; geometry collision cylinder length=0.13 radius=0.04; visual mesh filename=../../../model/HRP4c/graphics/R_WRIST_Y_rev2.obj
- link trunk: mass 18.9794300000 -> 12
- link trunk_rz: mass 18.9794300000 -> 1; geometry collision cylinder length=0.45 radius=0.13; visual mesh filename=../../../model/HRP4c/graphics/CHEST_Y2_rev2.obj

Commit message: up to date version from SRC

File: optitrack/model/HRP4c_green.urdf (robot description, URDF)
Before this commit: robot HRP4c, 39 links, 38 joints
Links:
- link neck_link2: geometry collision sphere radius=0.12; visual mesh filename=../../../model/HRP4c/graphics/Helmet_roboCop_rev2_green.obj

File: optitrack/model/HRP4c_purple.urdf (robot description, URDF)
Before this commit: robot HRP4c, 39 links, 38 joints
Links:
- link neck_link2: geometry collision sphere radius=0.12; visual mesh filename=../../../model/HRP4c/graphics/Helmet_roboCop_rev2_purple.obj
