Commit message: Post singularity update version

File: optitrack/model/HRP4c_purple.urdf (robot description, URDF)
Before this commit: robot HRP4c, 39 links, 38 joints
Joints:
- joint j10: limit lower=0.1 upper=2.5 effort=165 velocity=3.0718 -> lower=0.2 upper=2.5 effort=165 velocity=3.0718
- joint j4: limit lower=0.1 upper=2.5 effort=165 velocity=3.0718 -> lower=0.2 upper=2.5 effort=165 velocity=3.0718
